File: Electrical 23-24/ESC FPGA/fpga/fpgadocs.kicad_sch (KiCad schematic)
At the start: 0 parts

Commit message: idk but something
Other:
- added sheet UG393 (ug393.kicad_sch)
- added sheet UG394 (ug394.kicad_sch)
- note added: "PCB Design"
- note added: "Power Mngmt"
Changed lines of the file:
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@@
 (kicad_sch (version 20230121) (generator eeschema)
   (paper "A4")
+  (text "PCB Design" (at 86.36 97.79 0)
+    (effects (font (size 2.54 2.54)) (justify left bottom))
+  )
   (text "Configuration" (at 54.61 97.79 0)
     (effects (font (size 2.54 2.54)) (justify left bottom))
@@
   (text "Family\nOverview" (at 26.67 101.6 0)
     (effects (font (size 2.54 2.54)) (justify left bottom))
+  )
+  (text "Power Mngmt" (at 118.11 97.79 0)
+    (effects (font (size 2.54 2.54)) (justify left bottom))
+  )
+  (sheet (at 83.82 81.28) (size 31.75 33.02)
+    (stroke (width 0.1524) (type solid))
+    (fill (color 0 0 0 0.0000))
+    (property "Sheetname" "UG393" (at 85.09 85.09 0)
+      (effects (font (size 1.27 1.27)) (justify left bottom))
+    )
+    (property "Sheetfile" "ug393.kicad_sch" (at 85.09 111.76 0)
+      (effects (font (size 1.27 1.27)) (justify left top))
+    )
+    (instances
+      (project "fpga"
+        (path "/5bf59577-a814-4364-8f7a-37815cfb5474/bed8e914-c952-4392-8cc1-6131598d34ad" (page "13"))
+      )
+    )
   )
   (sheet (at 52.07 81.28) (size 31.75 33.02)
@@
       )
     )
+  )
+  (sheet (at 115.57 81.28) (size 31.75 33.02)
+    (stroke (width 0.1524) (type solid))
+    (fill (color 0 0 0 0.0000))
+    (property "Sheetname" "UG394" (at 116.84 85.09 0)
+      (effects (font (size 1.27 1.27)) (justify left bottom))
+    )
+    (property "Sheetfile" "ug394.kicad_sch" (at 116.84 111.76 0)
+      (effects (font (size 1.27 1.27)) (justify left top))
+    )
+    (instances
+      (project "fpga"
+        (path "/5bf59577-a814-4364-8f7a-37815cfb5474/bed8e914-c952-4392-8cc1-6131598d34ad" (page "14"))
+      )
+    )
