File: Electrical 23-24/ESC FPGA/fpga/qspi.kicad_sch (KiCad schematic)
At the start: 0 parts

Commit message: Add programmer
Parts:
- added U5: MT25QUxxxxxx1xW7, Package_SO:SOIC-8W_5.3x5.3mm_P1.27mm, symbol Memory_Flash:MT25QUxxxxxx1xW7
Connections:
- new net GND: U5.4 (VSS)
- new net SPI_CLK: U5.6 (C)
- new net SPI_CS: U5.1 (~{S})
- new net SPI_MISO1: U5.2 (DQ1)
- new net SPI_MISO2: U5.3 (~{W}/DQ2)
- new net SPI_MISO3: U5.7 (~{HOLD}/DQ3)
- new net SPI_MOSI/MISO0: U5.5 (DQ0)
- new net VCCO_2: U5.8 (VCC)
Other:
- note added: "Part: MT25QL128ABA1ESE-0SIT TR Digi: https://www.digikey.com/en/products/detail/micron-technology-inc/MT25QL128ABA1ESE-0SIT-TR/6595661 Datasheet: https://media-www.micron.com/-/media/client/global/documents/products/data-sheet/nor-flash/serial-nor/mt25q/die-rev-a/mt25q_qlhs_l_128_aba_0.pdf"
- note added: "Power-on in 0.3ms << 2ms"
Changed lines of the file:
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@@
 (kicad_sch (version 20230121) (generator eeschema)
   (paper "A4")
+  (text "Part: MT25QL128ABA1ESE-0SIT TR\nDigi: https://www.digikey.com/en/products/detail/micron-technology-inc/MT25QL128ABA1ESE-0SIT-TR/6595661\nDatasheet: https://media-www.micron.com/-/media/client/global/documents/products/data-sheet/nor-flash/serial-nor/mt25q/die-rev-a/mt25q_qlhs_l_128_aba_0.pdf"
+    (at 15.24 29.21 0)
+    (effects (font (size 2.54 2.54)) (justify left bottom))
+  )
+  (text "Power-on in 0.3ms << 2ms" (at 119.38 107.95 0)
+    (effects (font (size 1.27 1.27)) (justify left bottom))
+  )
+  (global_label "SPI_CLK" (shape input) (at 124.46 76.2 180) (fields_autoplaced)
+    (effects (font (size 1.27 1.27)) (justify right))
+    (property "Intersheetrefs" "${INTERSHEET_REFS}" (at 113.8548 76.2 0)
+      (effects (font (size 1.27 1.27)) (justify right) hide)
+    )
+  )
+  (global_label "SPI_MISO2" (shape input) (at 124.46 83.82 180) (fields_autoplaced)
+    (effects (font (size 1.27 1.27)) (justify right))
+    (property "Intersheetrefs" "${INTERSHEET_REFS}" (at 111.6172 83.82 0)
+      (effects (font (size 1.27 1.27)) (justify right) hide)
+    )
+  )
+  (global_label "SPI_CS" (shape input) (at 124.46 73.66 180) (fields_autoplaced)
+    (effects (font (size 1.27 1.27)) (justify right))
+    (property "Intersheetrefs" "${INTERSHEET_REFS}" (at 114.9434 73.66 0)
+      (effects (font (size 1.27 1.27)) (justify right) hide)
+    )
+  )
+  (global_label "VCCO_2" (shape input) (at 134.62 68.58 90) (fields_autoplaced)
+    (effects (font (size 1.27 1.27)) (justify left))
+    (property "Intersheetrefs" "${INTERSHEET_REFS}" (at 134.62 58.4586 90)
+      (effects (font (size 1.27 1.27)) (justify left) hide)
+    )
+  )
+  (global_label "SPI_MISO3" (shape input) (at 124.46 86.36 180) (fields_autoplaced)
+    (effects (font (size 1.27 1.27)) (justify right))
+    (property "Intersheetrefs" "${INTERSHEET_REFS}" (at 111.6172 86.36 0)
+      (effects (font (size 1.27 1.27)) (justify right) hide)
+    )
+  )
+  (global_label "SPI_MISO1" (shape input) (at 124.46 81.28 180) (fields_autoplaced)
+    (effects (font (size 1.27 1.27)) (justify right))
+    (property "Intersheetrefs" "${INTERSHEET_REFS}" (at 111.6172 81.28 0)
+      (effects (font (size 1.27 1.27)) (justify right) hide)
+    )
+  )
+  (global_label "SPI_MOSI{slash}MISO0" (shape input) (at 124.46 78.74 180) (fields_autoplaced)
+    (effects (font (size 1.27 1.27)) (justify right))
+    (property "Intersheetrefs" "${INTERSHEET_REFS}" (at 105.6905 78.74 0)
+      (effects (font (size 1.27 1.27)) (justify right) hide)
+    )
+  )
+  (symbol (lib_id "power:GND") (at 134.62 93.98 0) (unit 1)
+    (in_bom yes) (on_board yes) (dnp no) (fields_autoplaced)
+    (property "Reference" "#PWR08" (at 134.62 100.33 0)
+      (effects (font (size 1.27 1.27)) hide)
+    )
+    (property "Value" "GND" (at 134.62 99.06 0)
+      (effects (font (size 1.27 1.27)))
+    )
+    (property "Footprint" "" (at 134.62 93.98 0)
+      (effects (font (size 1.27 1.27)) hide)
+    )
+    (property "Datasheet" "" (at 134.62 93.98 0)
+      (effects (font (size 1.27 1.27)) hide)
+    )
+    (pin "1")
+    (instances
+      (project "fpga"
+        (path "/5bf59577-a814-4364-8f7a-37815cfb5474/edbd8098-adc9-4a81-8225-56e5824f7b8b"
+          (reference "#PWR08") (unit 1)
+        )
+      )
+    )
+  )
+  (symbol (lib_id "Memory_Flash:MT25QUxxxxxx1xW7") (at 134.62 81.28 0) (unit 1)
+    (in_bom yes) (on_board yes) (dnp no) (fields_autoplaced)
+    (property "Reference" "U5" (at 143.51 80.01 0)
+      (effects (font (size 1.27 1.27)) (justify left))
+    )
+    (property "Value" "MT25QUxxxxxx1xW7" (at 143.51 82.55 0)
+      (effects (font (size 1.27 1.27)) (justify left))
+    )
+    (property "Footprint" "Package_SO:SOIC-8W_5.3x5.3mm_P1.27mm" (at 154.94 78.74 0)
+      (effects (font (size 1.27 1.27)) hide)
+    )
+    (property "Datasheet" "https://media-www.micron.com/-/media/client/global/documents/products/data-sheet/nor-flash/serial-nor/mt25q/die-rev-a/mt25q_qljs_u_256_aba_0.pdf" (at 134.62 63.5 0)
+      (effects (font (size 1.27 1.27)) hide)
+    )
+    (pin "1")
+    (pin "2")
+    (pin "3")
+    (pin "4")
+    (pin "5")
+    (pin "6")
+    (pin "7")
+    (pin "8")
+    (instances
+      (project "fpga"
+        (path "/5bf59577-a814-4364-8f7a-37815cfb5474/edbd8098-adc9-4a81-8225-56e5824f7b8b"
+          (reference "U5") (unit 1)
+        )
+      )
+    )
+  )
 )

Commit message: idk but something
Parts:
- U5: value MT25QUxxxxxx1xW7 -> MT25QL128ABA1ESE; Digi (none) -> https://www.digikey.com/en/products/detail/micron-technolog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
Changed lines of the file:
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@@
       (effects (font (size 1.27 1.27)) (justify left))
     )
-    (property "Value" "MT25QUxxxxxx1xW7" (at 143.51 82.55 0)
+    (property "Value" "MT25QL128ABA1ESE" (at 143.51 82.55 0)
       (effects (font (size 1.27 1.27)) (justify left))
     )
@@
       (effects (font (size 1.27 1.27)) hide)
     )
-    (property "Datasheet" "https://media-www.micron.com/-/media/client/global/documents/products/data-sheet/nor-flash/serial-nor/mt25q/die-rev-a/mt25q_qljs_u_256_aba_0.pdf" (at 134.62 63.5 0)
+    (property "Datasheet" "https://media-www.micron.com/-/media/client/global/documents/products/data-sheet/nor-flash/serial-nor/mt25q/die-rev-a/mt25q_qlhs_l_128_aba_0.pdf" (at 134.62 63.5 0)
       (effects (font (size 1.27 1.27)) hide)
     )
+    (property "Digi" "https://www.digikey.com/en/products/detail/micron-technology-inc/MT25QL128ABA1ESE-0SIT-TR/6595661" (at 134.62 81.28 0)
+      (effects (font (size 1.27 1.27)) hide)
+    )

Commit message: Add fpga stuff and stencils
Changed lines of the file:
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@@
+    )
+  )
+  (global_label "GND" (shape input) (at 270.51 50.8 90) (fields_autoplaced)
+    (effects (font (size 1.27 1.27)) (justify left))
+    (property "Intersheetrefs" "${INTERSHEET_REFS}" (at 270.51 43.9443 90)
+      (effects (font (size 1.27 1.27)) (justify left) hide)
     )
   )
@@
     )
   )
+  (symbol (lib_id "power:GND") (at 270.51 50.8 0) (unit 1)
+    (in_bom yes) (on_board yes) (dnp no) (fields_autoplaced)
+    (property "Reference" "#PWR016" (at 270.51 57.15 0)
+      (effects (font (size 1.27 1.27)) hide)
+    )
+    (property "Value" "GND" (at 270.51 55.88 0)
+      (effects (font (size 1.27 1.27)))
+    )
+    (property "Footprint" "" (at 270.51 50.8 0)
+      (effects (font (size 1.27 1.27)) hide)
+    )
+    (property "Datasheet" "" (at 270.51 50.8 0)
+      (effects (font (size 1.27 1.27)) hide)
+    )
+    (pin "1")
+    (instances
+      (project "fpga"
+        (path "/5bf59577-a814-4364-8f7a-37815cfb5474/3e04db34-3f8a-4742-be82-6fa24c009343"
+          (reference "#PWR016") (unit 1)
+        )
+        (path "/5bf59577-a814-4364-8f7a-37815cfb5474/1f83b38b-56ef-4110-879b-13379f9dd920"
+          (reference "#PWR026") (unit 1)
+        )
+        (path "/5bf59577-a814-4364-8f7a-37815cfb5474/a286b274-4434-47ab-983d-e64806fdcbd6"
+          (reference "#PWR036") (unit 1)
+        )
+        (path "/5bf59577-a814-4364-8f7a-37815cfb5474/edbd8098-adc9-4a81-8225-56e5824f7b8b"
+          (reference "#PWR038") (unit 1)
+        )
+      )
+    )
+  )
