File: Electrical 23-24/ESC FPGA/fpga/bank2.kicad_sch (KiCad schematic)
At the start: 18 parts, among them U1 XC6SLX4-TQG144, X1 KC5032Z100.000C1JX00

Commit message: Finished FPGA board schematic
Parts:
- added LED1, LED2, LED3, LED4: B38G3RGB-10D0003H2U1930, B38G3RGB-10D0003H2U1930_HVK, symbol fpga:B38G3RGB-10D0003H2U1930
- added R35, R36, R37, R44: 270, symbol Device:R
- added R38, R39, R40, R41, R42, R43, R45, R46: 56, symbol Device:R
- added R47, R48, R49, R50, R51, R52: 1k, symbol Device:R
- added R53, R54, R55, R56, R57, R58: 10k, symbol Device:R
- added SW1: SW_SPDT, symbol Switch:SW_SPDT
- added SW10, SW11, SW9: SW_SPST, symbol Switch:SW_SPST
- added SW6, SW7, SW8: SW_Push, symbol Switch:SW_Push
- added U14: FXMA108BQX, WQFN20_2P5X4P5_ONS, symbol fpga:FXMA108BQX
Connections:
- net 3V3: now also SW1.3 (C), U14.1 (VCCA)
- net GND: now also R53.1, R54.1, R55.1, R56.1, R57.1, R58.1, U14.10 (GND)
- net VCCO_2: now also LED1.3, LED2.3, LED3.3, LED4.3, R47.2, R48.2, R49.2, R50.2
- net VCCO_3: now also R51.2, R52.2
- net PMOD2_7: now reaches U1.1 (IO_L83N_VREF_3)
- net PMOD2_0: now reaches U1.10 (IO_L50P_3)
- net PMOD1_7: now reaches U1.11 (IO_L49N_3)
- net PMOD1_3: now reaches U1.12 (IO_L49P_3)
- net PMOD1_6: now reaches U1.14 (IO_L44N_GCLK20_3)
- net PMOD1_5: now reaches U1.15 (IO_L44P_GCLK21_3)
- net PMOD1_4: now reaches U1.16 (IO_L43N_GCLK22_IRDY2_3)
- net PMOD1_2: now reaches U1.17 (IO_L43P_GCLK23_3)
- net PMOD2_6: now reaches U1.2 (IO_L83P_3)
- net PMOD1_1: now reaches U1.21 (IO_L42N_GCLK24_3)
- net PMOD1_0: now reaches U1.22 (IO_L42P_GCLK25_TRDY2_3)
- net at U1.23 (IO_L41N_GCLK26_3): now also U14.9 (A7)
- net at U1.24 (IO_L41P_GCLK27_3): now also U14.8 (A6)
- net at U1.26 (IO_L37N_3): now also U14.7 (A5)
- net at U1.27 (IO_L37P_3): now also U14.6 (A4)
- net at U1.29 (IO_L36N_3): now also U14.5 (A3)
- net at U1.30 (IO_L36P_3): now also U14.4 (A2)
- net at U1.32 (IO_L2N_3): now also U14.3 (A1)
- net at U1.33 (IO_L2P_3): now also U14.2 (A0)
- net SW3: now reaches U1.34 (IO_L1N_VREF_3)
- net SW3: now also R58.2, SW11.1 (A)
- net SW2: now reaches U1.35 (IO_L1P_3)
- net SW2: now also R57.2, SW10.1 (A)
- net R1: now reaches U1.40 (IO_L64N_D9_2)
- net R1: now also R35.2
- net G1: now reaches U1.41 (IO_L64P_D8_2)
- net G1: now also R38.2
- net B1: now reaches U1.43 (IO_L62N_D6_2)
- net B1: now also R39.2
- net R2: now reaches U1.44 (IO_L62P_D5_2)
- net R2: now also R36.2
- net G2: now reaches U1.45 (IO_L49N_D4_2)
- net G2: now also R40.2
- net B2: now reaches U1.46 (IO_L49P_D3_2)
- net B2: now also R41.2
- net R3: now reaches U1.47 (IO_L48N_RDWR_B_VREF_2)
- net R3: now also R37.2
- net G3: now reaches U1.48 (IO_L48P_D7_2)
- net G3: now also R42.2
- net PMOD2_5: now reaches U1.5 (IO_L52N_3)
- net B3: now reaches U1.50 (IO_L31N_GCLK30_D15_2)
- net B3: now also R43.2
- net BTN1: now reaches U1.51 (IO_L31P_GCLK31_D14_2)
- net BTN1: now also R53.2, SW6.1
- net BTN2: now reaches U1.56 (IO_L30P_GCLK1_D13_2)
- net BTN2: now also R54.2, SW7.1
- net R4: now reaches U1.57 (IO_L14N_D12_2)
- net R4: now also R44.2
- net G4: now reaches U1.58 (IO_L14P_D11_2)
- net G4: now also R45.2
- net B4: now reaches U1.59 (IO_L13N_D10_2)
- net B4: now also R46.2
- net PMOD2_4: now reaches U1.6 (IO_L52P_3)
- net BTN3: now reaches U1.66 (IO_L2N_CMPMOSI_2)
- net BTN3: now also R55.2, SW8.1
- net SW1: now reaches U1.67 (IO_L2P_CMPCLK_2)
- net SW1: now also R56.2, SW9.1 (A)
- net PMOD2_3: now reaches U1.7 (IO_L51N_3)
- net PMOD2_2: now reaches U1.8 (IO_L51P_3)
- net PMOD2_1: now reaches U1.9 (IO_L50N_3)
- new net: LED3.1, R42.1
- new net: R51.1, SW10.2 (B)
- new net: LED2.1, R40.1
- new net: LED2.2, R41.1
- new net: LED2.4, R36.1
- new net: LED4.2, R46.1
- new net: R50.1, SW9.2 (B)
- new net: R52.1, SW11.2 (B)
- new net: LED1.1, R38.1
- new net: R47.1, SW6.2
- new net: LED1.4, R35.1
- new net: SW1.2 (B), U14.20 (VCCB)
- new net: LED3.2, R43.1
- new net: LED3.4, R37.1
- new net: LED4.1, R45.1
- new net: R49.1, SW8.2
- new net: LED4.4, R44.1
- new net: R48.1, SW7.2
- new net: LED1.2, R39.1
- new net GPIO16: U14.19 (B0)
- new net GPIO17: U14.18 (B1)
- new net GPIO18: U14.12 (B7)
- new net GPIO19: U14.16 (B3)
- new net GPIO20: U14.15 (B4)
- new net GPIO21: U14.14 (B5)
- new net GPIO22: U14.13 (B6)
- new net GPIO23: U14.17 (B2)
- new net OE: U14.11 (/OE)
- new net VUSB: SW1.1 (A)
- no-connect marks 0 -> 1
Other:
- note added: "2 PMOD: 16 Pins 3 Switches: 3 Pins 3 Buttons: 3 Pins 4 RGB: 12 Pins Total: 34 Pins Have: 34 Pins"
- note added: "2V Vf Red 3V Vf Green/Blue 5mA Current"
- note added: "Level Shifters"
- note added: "Pending: 8 switches (dip switch) rgb led 1 led per button Done: Board-to-Board (PHY) Level Shifter/GPIO 2 PMOD Won't Do: HDMI"
- note removed: "4 pmod 8 switches (dip switch) gpio (raspi header or arduino shield) rgb led 1 led per button level shifter? -----HDMI Board-to-Board (PHY)"
- moved on the sheet: C52, C6, R10, R11, R12, R13, R14, R5, R6, R7, R8, U1B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

Commit message: Made BOM, need to modify footprints
Parts:
- removed SW1: SW_SPDT, symbol Switch:SW_SPDT
- removed SW10, SW11, SW9: SW_SPST, symbol Switch:SW_SPST
- removed SW6, SW7, SW8: SW_Push, symbol Switch:SW_Push
- removed U1: XC6SLX4-TQG144, symbol FPGA_Xilinx_Spartan6:XC6SLX4-TQG144
- added SW1 (x4): SW_SPDT, Connector_PinHeader_2.54mm:PinHeader_1x03_P2.54mm_Vertical, symbol Switch:SW_SPDT
- added SW2 (x3): SW_Push, fpga:NCA1, symbol Switch:SW_Push
- added U16: XC6SLX9-TQG144, fpga:TQFP-144_20x20mm_P0.5mm, symbol FPGA_Xilinx_Spartan6:XC6SLX9-TQG144
- C52: footprint Capacitor_SMD:C_0603_1608Metric_Pad1.08x0.95mm_HandSolder -> Capacitor_SMD:C_0402_1005Metric_Pad0.74x0.62mm_HandSolder
- C6: value u47 -> 0.47u; footprint (none) -> Capacitor_SMD:C_0402_1005Metric_Pad0.74x0.62mm_HandSolder
- C6: value 4u7 -> 4.7u; footprint (none) -> Capacitor_SMD:C_0402_1005Metric_Pad0.74x0.62mm_HandSolder
- LED1, LED2, LED3, LED4: footprint B38G3RGB-10D0003H2U1930_HVK -> fpga:B38G3RGB-10D0003H2U1930_HVK; Digi (none) -> https://www.digikey.com/en/products/detail/harvatek-corpora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
- R10, R11, R13, R14, R35, R36, R37, R38, R39, R40, R41, R42, R43, R44, R45, R46, R47, R48, R49, R50, R51, R52, R53, R54, R55, R56, R57, R58, R7, R8: footprint (none) -> Resistor_SMD:R_0402_1005Metric_Pad0.72x0.64mm_HandSolder
- R12: value 10 -> 2.2; footprint (none) -> Resistor_SMD:R_0402_1005Metric_Pad0.72x0.64mm_HandSolder
- R5: value 4k7 -> 4.7k; footprint (none) -> Resistor_SMD:R_0402_1005Metric_Pad0.72x0.64mm_HandSolder
- R6: value 2k4 -> 2.2k; footprint (none) -> Resistor_SMD:R_0402_1005Metric_Pad0.72x0.64mm_HandSolder
- U14: footprint WQFN20_2P5X4P5_ONS -> fpga:WQFN20_2P5X4P5_ONS
Connections:
- net 3V3: now also SW1.3 (C)
- net B1: now also U16.43 (IO_L62N_D6_2)
- net B2: now also U16.46 (IO_L49P_D3_2)
- net B3: now also U16.50 (IO_L31N_GCLK30_D15_2)
- net B4: now also U16.59 (IO_L13N_D10_2)
- net BTN1: now also SW2.1, U16.51 (IO_L31P_GCLK31_D14_2)
- net BTN2: now also SW2.1, U16.56 (IO_L30P_GCLK1_D13_2)
- net BTN3: now also SW2.1, U16.66 (IO_L2N_CMPMOSI_2)
- net G1: now also U16.41 (IO_L64P_D8_2)
- net G2: now also U16.45 (IO_L49N_D4_2)
- net G3: now also U16.48 (IO_L48P_D7_2)
- net G4: now also U16.58 (IO_L14P_D11_2)
- net INIT_B_IO: now also U16.39 (IO_L65P_INIT_B_2)
- net M0_IO: now also U16.69 (IO_L1N_M0_CMPMISO_2)
- net M1_IO: now also U16.60 (IO_L13P_M1_2)
- net OSCI: now also U16.55 (IO_L30N_GCLK0_USERCCLK_2)
- net PMOD1_0: now also U16.22 (IO_L42P_GCLK25_TRDY2_3)
- net PMOD1_1: now also U16.21 (IO_L42N_GCLK24_3)
- net PMOD1_2: now also U16.17 (IO_L43P_GCLK23_3)
- net PMOD1_3: now also U16.12 (IO_L49P_3)
- net PMOD1_4: now also U16.16 (IO_L43N_GCLK22_IRDY2_3)
- net PMOD1_5: now also U16.15 (IO_L44P_GCLK21_3)
- net PMOD1_6: now also U16.14 (IO_L44N_GCLK20_3)
- net PMOD1_7: now also U16.11 (IO_L49N_3)
- net PMOD2_0: now also U16.10 (IO_L50P_3)
- net PMOD2_1: now also U16.9 (IO_L50N_3)
- net PMOD2_2: now also U16.8 (IO_L51P_3)
- net PMOD2_3: now also U16.7 (IO_L51N_3)
- net PMOD2_4: now also U16.6 (IO_L52P_3)
- net PMOD2_5: now also U16.5 (IO_L52N_3)
- net PMOD2_6: now also U16.2 (IO_L83P_3)
- net PMOD2_7: now also U16.1 (IO_L83N_VREF_3)
- net R1: now also U16.40 (IO_L64N_D9_2)
- net R2: now also U16.44 (IO_L62P_D5_2)
- net R3: now also U16.47 (IO_L48N_RDWR_B_VREF_2)
- net R4: now also U16.57 (IO_L14N_D12_2)
- net SPI_CLK: now also U16.70 (IO_L1P_CCLK_2)
- net SPI_CS: now also U16.38 (IO_L65N_CSO_B_2)
- net SPI_MISO1_IO: now also U16.65 (IO_L3P_D0_DIN_MISO_MISO1_2)
- net SPI_MISO2: now also U16.62 (IO_L12P_D1_MISO2_2)
- net SPI_MISO3: now also U16.61 (IO_L12N_D2_MISO3_2)
- net SPI_MOSI/MISO0: now also U16.64 (IO_L3N_MOSI_CSI_B_MISO0_2)
- net SW1: now also SW1.2 (B), U16.67 (IO_L2P_CMPCLK_2)
- net SW2: now also SW1.2 (B), U16.35 (IO_L1P_3)
- net SW3: now also SW1.2 (B), U16.34 (IO_L1N_VREF_3)
- net VCCO_2: now also U16.42 (VCCO_2), U16.63 (VCCO_2)
- net VCCO_3: now also U16.18 (VCCO_3), U16.31 (VCCO_3), U16.4 (VCCO_3)
- net VUSB: now also SW1.1 (A)
- net at R51.1: now also SW1.3 (C)
- net at R50.1: now also SW1.3 (C)
- net at R52.1: now also SW1.3 (C)
- net at R47.1: now also SW2.2
- net at U14.20 (VCCB): now also SW1.2 (B)
- net at R49.1: now also SW2.2
- net at R48.1: now also SW2.2
- net at U14.9 (A7): now also U16.23 (IO_L41N_GCLK26_3)
- net at U14.8 (A6): now also U16.24 (IO_L41P_GCLK27_3)
- net at U14.7 (A5): now also U16.26 (IO_L37N_3)
- net at U14.6 (A4): now also U16.27 (IO_L37P_3)
- net at U14.5 (A3): now also U16.29 (IO_L36N_3)
- net at U14.4 (A2): now also U16.30 (IO_L36P_3)
- net at U14.3 (A1): now also U16.32 (IO_L2N_3)
- net at U14.2 (A0): now also U16.33 (IO_L2P_3)
- no-connect marks 1 -> 4
Other:
- moved on the sheet: R50, R51, R52
