File: Electrical 23-24/Power Distribution Board/pw_protection.kicad_sch (KiCad schematic)
At the start: 6 parts, among them Q201 PNP, Q202 PNP

Commit message: Finalize PDB board
Parts:
- D201: value 4.5V -> 5.1V; footprint Aero_PDB:SODFL1608X70N -> Aero_PDB:SOD1608X70; Digi (none) -> https://www.digikey.com/en/products/detail/onsemi/MM5Z5V1T1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
Connections:
- net RPI_PWR_IN: now also Q201.3 (E), Q202.3 (E)
Changed lines of the file:
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@@
   (junction (at 99.06 82.55) (diameter 0) (color 0 0 0 0)
   )
+  (junction (at 138.43 48.26) (diameter 0) (color 0 0 0 0)
+  )
+  (junction (at 114.3 53.34) (diameter 0) (color 0 0 0 0)
+  )
   (wire (pts (xy 99.06 82.55) (xy 138.43 82.55))
     (stroke (width 0) (type default))
@@
   )
   (wire (pts (xy 138.43 49.53) (xy 138.43 48.26))
+    (stroke (width 0) (type default))
+  )
+  (wire (pts (xy 114.3 48.26) (xy 114.3 53.34))
+    (stroke (width 0) (type default))
+  )
+  (wire (pts (xy 138.43 48.26) (xy 114.3 48.26))
     (stroke (width 0) (type default))
   )
@@
       (effects (font (size 1.27 1.27)) hide)
     )
+    (pin "1")
+    (pin "2")
     (pin "3")
-    (pin "2")
-    (pin "1")
     (instances
       (project "Aero_PDB"
@@
       (effects (font (size 1.27 1.27)) hide)
     )
-    (pin "2")
-    (pin "1")
+    (pin "1")
+    (pin "2")
     (instances
       (project "Aero_PDB"
@@
       (effects (font (size 1.27 1.27)) hide)
     )
+    (pin "1")
+    (pin "2")
     (pin "3")
-    (pin "2")
-    (pin "1")
     (instances
       (project "Aero_PDB"
@@
       (effects (font (size 1.27 1.27)) hide)
     )
-    (pin "2")
-    (pin "1")
+    (pin "1")
+    (pin "2")
     (instances
       (project "Aero_PDB"
@@
       (effects (font (size 1.27 1.27)) hide)
     )
-    (pin "2")
-    (pin "1")
+    (pin "1")
+    (pin "2")
     (instances
       (project "Aero_PDB"
@@
       (effects (font (size 1.27 1.27)) (justify left))
     )
-    (property "Value" "4.5V " (at 140.97 76.2 90)
-      (effects (font (size 1.27 1.27)) (justify left))
-    )
-    (property "Footprint" "Aero_PDB:SODFL1608X70N" (at 138.43 74.93 0)
-      (effects (font (size 1.27 1.27)) hide)
-    )
-    (property "Datasheet" "~" (at 138.43 74.93 0)
-      (effects (font (size 1.27 1.27)) hide)
-    )
+    (property "Value" "5.1V" (at 140.97 76.2 90)
+      (effects (font (size 1.27 1.27)) (justify left))
+    )
+    (property "Footprint" "Aero_PDB:SOD1608X70" (at 138.43 74.93 0)
+      (effects (font (size 1.27 1.27)) hide)
+    )
+    (property "Datasheet" "https://www.onsemi.com/pdf/datasheet/mm5z2v4t1-d.pdf" (at 138.43 74.93 0)
+      (effects (font (size 1.27 1.27)) hide)
+    )
+    (property "Digi" "https://www.digikey.com/en/products/detail/onsemi/MM5Z5V1T1G/921103" (at 138.43 74.93 90)
+      (effects (font (size 1.27 1.27)) hide)
+    )
