File: Electrical 23-24/Power Distribution Board/Aero_PDB.kicad_sch (KiCad schematic)
At the start: 21 parts, among them J1 Conn_01x04_Pin, J101 Gimbal Conn, J102 Pixhawk Servo Conn, J103 Pixawk Backup Power, J104 USB_OTG, J105 Servo to PDB Conn, J106 JST_XH_4, J107 DCJ200-10-A-XX-K_REVA, J108 JST_XH_4, J2 Conn_01x04_Pin, J3 RCIN, J4 RCIN

Commit message: Changed USB micro to USB A
Parts:
- removed J104: USB_OTG, Aero_PDB:MOLEX_47346-0001, symbol Connector:USB_OTG
- added J113: USB_A, Aero_PDB:GCT_USB1130-15-A_REVA, symbol Connector:USB_A
- renumbered J107 to J106, J3 to J107, J106 to J109, J4 to J110, J1 to J111, J2 to J112
Connections:
- net GND: now also J113.4 (GND)
- net RPI_PWR: now also J113.1 (VBUS)
Changed lines of the file:
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@@
   )
   (no_connect (at 123.19 123.19))
+  (no_connect (at 133.35 130.81))
   (no_connect (at 207.01 144.78))
   (no_connect (at 233.68 144.78))
   (no_connect (at 111.76 83.82))
   (no_connect (at 123.19 120.65))
-  (no_connect (at 123.19 125.73))
   (wire (pts (xy 53.34 132.08) (xy 50.8 132.08))
     (stroke (width 0) (type default))
@@
   (symbol (lib_id "Connector:Conn_01x03_Socket") (at 212.09 144.78 0) (unit 1)
     (in_bom yes) (on_board yes) (dnp no)
-    (property "Reference" "J3" (at 205.74 135.89 0)
+    (property "Reference" "J107" (at 205.74 135.89 0)
       (effects (font (size 1.27 1.27)) (justify left))
     )
@@
       (project "Aero_PDB"
         (path "/ec3864f8-beea-4bd9-8117-4ec49632e630"
-          (reference "J3") (unit 1)
+          (reference "J107") (unit 1)
         )
       )
@@
   (symbol (lib_id "Connector:Conn_01x04_Pin") (at 217.17 90.17 0) (mirror y) (unit 1)
     (in_bom yes) (on_board yes) (dnp no)
-    (property "Reference" "J106" (at 210.82 80.01 0)
+    (property "Reference" "J109" (at 210.82 80.01 0)
       (effects (font (size 1.27 1.27)))
     )
@@
       (project "Aero_PDB"
         (path "/ec3864f8-beea-4bd9-8117-4ec49632e630"
-          (reference "J106") (unit 1)
+          (reference "J109") (unit 1)
+        )
+      )
+    )
+  )
+  (symbol (lib_id "Connector:USB_A") (at 130.81 120.65 0) (mirror y) (unit 1)
+    (in_bom yes) (on_board yes) (dnp no)
+    (property "Reference" "J113" (at 128.27 107.95 0)
+      (effects (font (size 1.27 1.27)) (justify right))
+    )
+    (property "Value" "USB_A" (at 128.27 110.49 0)
+      (effects (font (size 1.27 1.27)) (justify right))
+    )
+    (property "Footprint" "Aero_PDB:GCT_USB1130-15-A_REVA" (at 127 121.92 0)
+      (effects (font (size 1.27 1.27)) hide)
+    )
+    (property "Datasheet" " ~" (at 127 121.92 0)
+      (effects (font (size 1.27 1.27)) hide)
+    )
+    (pin "1")
+    (pin "2")
+    (pin "4")
+    (pin "5")
+    (pin "3")
+    (instances
+      (project "Aero_PDB"
+        (path "/ec3864f8-beea-4bd9-8117-4ec49632e630"
+          (reference "J113") (unit 1)
         )
       )
@@
   (symbol (lib_id "power:GND") (at 233.68 147.32 0) (unit 1)
     (in_bom yes) (on_board yes) (dnp no) (fields_autoplaced)
-    (property "Reference" "#PWR02" (at 233.68 153.67 0)
+    (property "Reference" "#PWR0122" (at 233.68 153.67 0)
       (effects (font (size 1.27 1.27)) hide)
     )
@@
       (project "Aero_PDB"
         (path "/ec3864f8-beea-4bd9-8117-4ec49632e630"
-          (reference "#PWR02") (unit 1)
+          (reference "#PWR0122") (unit 1)
         )
       )
@@
   (symbol (lib_id "power:GND") (at 109.22 88.9 0) (unit 1)
     (in_bom yes) (on_board yes) (dnp no) (fields_autoplaced)
-    (property "Reference" "#PWR03" (at 109.22 95.25 0)
+    (property "Reference" "#PWR0116" (at 109.22 95.25 0)
       (effects (font (size 1.27 1.27)) hide)
     )
@@
       (project "Aero_PDB"
         (path "/ec3864f8-beea-4bd9-8117-4ec49632e630"
-          (reference "#PWR03") (unit 1)
+          (reference "#PWR0116") (unit 1)
         )
       )
@@
     )
   )
-  (symbol (lib_id "Connector:USB_OTG") (at 130.81 120.65 0) (mirror y) (unit 1)
-    (in_bom yes) (on_board yes) (dnp no)
-    (property "Reference" "J104" (at 130.81 107.95 0)
-      (effects (font (size 1.27 1.27)))
-    )
-    (property "Value" "USB_OTG" (at 130.81 110.49 0)
-      (effects (font (size 1.27 1.27)))
-    )
-    (property "Footprint" "Aero_PDB:MOLEX_47346-0001" (at 127 121.92 0)
-      (effects (font (size 1.27 1.27)) hide)
-    )
-    (property "Datasheet" " ~" (at 127 121.92 0)
-      (effects (font (size 1.27 1.27)) hide)
-    )
-    (pin "1")
-    (pin "2")
-    (pin "3")
-    (pin "4")
-    (pin "5")
-    (instances
-      (project "Aero_PDB"
-        (path "/ec3864f8-beea-4bd9-8117-4ec49632e630"
-          (reference "J104") (unit 1)
-        )
-      )
-    )
-  )
   (symbol (lib_id "power:GND") (at 53.34 162.56 0) (unit 1)
     (in_bom yes) (on_board yes) (dnp no) (fields_autoplaced)
@@
   (symbol (lib_id "Connector:Conn_01x03_Socket") (at 238.76 144.78 0) (unit 1)
     (in_bom yes) (on_board yes) (dnp no)
-    (property "Reference" "J4" (at 232.41 135.89 0)
+    (property "Reference" "J110" (at 232.41 135.89 0)
       (effects (font (size 1.27 1.27)) (justify left))
     )
@@
       (project "Aero_PDB"
         (path "/ec3864f8-beea-4bd9-8117-4ec49632e630"
-          (reference "J4") (unit 1)
+          (reference "J110") (unit 1)
         )
       )
@@
   (symbol (lib_id "Aero_PDB_parts:DCJ200-10-A-XX-K_REVA") (at 158.75 124.46 0) (mirror y) (unit 1)
     (in_bom yes) (on_board yes) (dnp no)
-    (property "Reference" "J107" (at 161.9858 115.57 0)
+    (property "Reference" "J106" (at 161.9858 115.57 0)
       (effects (font (size 1.27 1.27)))
     )
@@
       (project "Aero_PDB"
         (path "/ec3864f8-beea-4bd9-8117-4ec49632e630"
-          (reference "J107") (unit 1)
+          (reference "J106") (unit 1)
         )
       )
@@
   (symbol (lib_id "Connector:Conn_01x04_Pin") (at 245.11 90.17 0) (mirror y) (unit 1)
     (in_bom yes) (on_board yes) (dnp no)
-    (property "Reference" "J2" (at 238.76 80.01 0)
+    (property "Reference" "J112" (at 238.76 80.01 0)
       (effects (font (size 1.27 1.27)))
     )
@@
       (project "Aero_PDB"
         (path "/ec3864f8-beea-4bd9-8117-4ec49632e630"
-          (reference "J2") (unit 1)
+          (reference "J112") (unit 1)
         )
       )
@@
   (symbol (lib_id "Connector:Conn_01x04_Pin") (at 243.84 113.03 0) (mirror y) (unit 1)
     (in_bom yes) (on_board yes) (dnp no)
-    (property "Reference" "J1" (at 237.49 102.87 0)
+    (property "Reference" "J111" (at 237.49 102.87 0)
       (effects (font (size 1.27 1.27)))
     )
@@
       (project "Aero_PDB"
         (path "/ec3864f8-beea-4bd9-8117-4ec49632e630"
-          (reference "J1") (unit 1)
+          (reference "J111") (unit 1)
         )
       )
@@
   (symbol (lib_name "GND_3") (lib_id "power:GND") (at 227.33 38.1 0) (unit 1)
     (in_bom yes) (on_board yes) (dnp no)
-    (property "Reference" "#PWR0120" (at 227.33 44.45 0)
+    (property "Reference" "#PWR0121" (at 227.33 44.45 0)
       (effects (font (size 1.27 1.27)) hide)
     )
@@
       (project "Aero_PDB"
         (path "/ec3864f8-beea-4bd9-8117-4ec49632e630"
-          (reference "#PWR0120") (unit 1)
+          (reference "#PWR0121") (unit 1)
         )
       )
@@
   (symbol (lib_id "power:GND") (at 207.01 147.32 0) (unit 1)
     (in_bom yes) (on_board yes) (dnp no) (fields_autoplaced)
-    (property "Reference" "#PWR01" (at 207.01 153.67 0)
+    (property "Reference" "#PWR0120" (at 207.01 153.67 0)
       (effects (font (size 1.27 1.27)) hide)
     )
@@
       (project "Aero_PDB"
         (path "/ec3864f8-beea-4bd9-8117-4ec49632e630"
-          (reference "#PWR01") (unit 1)
-        )
-      )
+          (reference "#PWR0120") (unit 1)
+        )
+      )
