File: Electrical 23-24/ESC FPGA/programmer/programmer.kicad_pcb (KiCad board)
At the start: 2 copper layers, 45.3 x 37.1 mm, 43 parts, among them J1 USB_B_Micro, J2 SFH11-PBPC-D07-ST-BK, J3 Conn_01x05_Pin, J5 Conn_02x8_Pin, J6 Conn_02x8_Pin, SW1 SW_DPST, U1 93C46C, U2 AMS1117-3.3, U3 NUP2202, U4 FT2232HL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

Commit message: Final board exports
Other:
- outline, holes or cut-outs redrawn
Changed lines of the file:
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@@
       (plot_on_all_layers_selection 0x0000000_00000000)
       (disableapertmacros false)
-      (usegerberextensions false)
-      (usegerberattributes true)
-      (usegerberadvancedattributes true)
-      (creategerberjobfile true)
+      (usegerberextensions true)
+      (usegerberattributes false)
+      (usegerberadvancedattributes false)
+      (creategerberjobfile false)
       (dashed_line_dash_ratio 12.000000)
       (dashed_line_gap_ratio 3.000000)
@@
       (psa4output false)
       (plotreference true)
-      (plotvalue true)
+      (plotvalue false)
       (plotinvisibletext false)
       (sketchpadsonfab false)
-      (subtractmaskfromsilk false)
+      (subtractmaskfromsilk true)
       (outputformat 1)
       (mirror false)
-      (drillshape 1)
+      (drillshape 0)
       (scaleselection 1)
-      (outputdirectory "")
+      (outputdirectory "jlc_exports/")
     )
   )
@@
   (gr_rect (start 160.6 102.2) (end 182 108.4)
     (stroke (width 0.15) (type default)) (fill none) (layer "Dwgs.User"))
-  (gr_line (start 97 62.9) (end 135.6 62.9)
+  (gr_line (start 98 62.9) (end 134.6 62.9)
     (stroke (width 0.1) (type default)) (layer "Edge.Cuts"))
-  (gr_line (start 97 100) (end 97 62.9)
+  (gr_line (start 97 99) (end 97 63.9)
     (stroke (width 0.1) (type default)) (layer "Edge.Cuts"))
-  (gr_line (start 142.3 88.6) (end 135.4 88.6)
+  (gr_line (start 141.3 88.6) (end 136.4 88.6)
     (stroke (width 0.1) (type default)) (layer "Edge.Cuts"))
-  (gr_line (start 135.6 62.9) (end 135.6 74.5)
+  (gr_arc (start 142.3 87.6) (mid 142.007107 88.307107) (end 141.3 88.6)
     (stroke (width 0.1) (type default)) (layer "Edge.Cuts"))
-  (gr_line (start 135.6 74.5) (end 142.3 74.5)
+  (gr_arc (start 136.6 74.5) (mid 135.892893 74.207107) (end 135.6 73.5)
     (stroke (width 0.1) (type default)) (layer "Edge.Cuts"))
-  (gr_line (start 142.3 74.5) (end 142.3 88.6)
+  (gr_line (start 135.6 63.9) (end 135.6 73.5)
     (stroke (width 0.1) (type default)) (layer "Edge.Cuts"))
-  (gr_line (start 135.4 88.6) (end 135.4 92.8)
+  (gr_line (start 136.6 74.5) (end 141.3 74.5)
     (stroke (width 0.1) (type default)) (layer "Edge.Cuts"))
-  (gr_line (start 135.4 92.8) (end 120.4 92.8)
+  (gr_arc (start 120.4 99) (mid 120.107107 99.707107) (end 119.4 100)
     (stroke (width 0.1) (type default)) (layer "Edge.Cuts"))
-  (gr_line (start 120.4 100) (end 97 100)
+  (gr_arc (start 134.6 62.9) (mid 135.307107 63.192893) (end 135.6 63.9)
     (stroke (width 0.1) (type default)) (layer "Edge.Cuts"))
-  (gr_line (start 120.4 92.8) (end 120.4 100)
+  (gr_line (start 142.3 75.5) (end 142.3 87.6)
+    (stroke (width 0.1) (type default)) (layer "Edge.Cuts"))
+  (gr_arc (start 135.4 91.8) (mid 135.107107 92.507107) (end 134.4 92.8)
+    (stroke (width 0.1) (type default)) (layer "Edge.Cuts"))
+  (gr_arc (start 135.4 89.6) (mid 135.692893 88.892893) (end 136.4 88.6)
+    (stroke (width 0.1) (type default)) (layer "Edge.Cuts"))
+  (gr_arc (start 97 63.9) (mid 97.292893 63.192893) (end 98 62.9)
+    (stroke (width 0.1) (type default)) (layer "Edge.Cuts"))
+  (gr_line (start 135.4 89.6) (end 135.4 91.8)
+    (stroke (width 0.1) (type default)) (layer "Edge.Cuts"))
+  (gr_line (start 134.4 92.8) (end 121.4 92.8)
+    (stroke (width 0.1) (type default)) (layer "Edge.Cuts"))
+  (gr_line (start 119.4 100) (end 98 100)
+    (stroke (width 0.1) (type default)) (layer "Edge.Cuts"))
+  (gr_arc (start 141.3 74.5) (mid 142.007107 74.792893) (end 142.3 75.5)
+    (stroke (width 0.1) (type default)) (layer "Edge.Cuts"))
+  (gr_line (start 120.4 93.8) (end 120.4 99)
+    (stroke (width 0.1) (type default)) (layer "Edge.Cuts"))
+  (gr_arc (start 120.4 93.8) (mid 120.692893 93.092893) (end 121.4 92.8)
+    (stroke (width 0.1) (type default)) (layer "Edge.Cuts"))
+  (gr_arc (start 98 100) (mid 97.292893 99.707107) (end 97 99)
     (stroke (width 0.1) (type default)) (layer "Edge.Cuts"))
   (gr_text "H4" (at 121.8 92.5) (layer "B.SilkS")
