File: Electrical 24-25/Logan/Servo Tester/servo_tester.kicad_pcb (KiCad board)
At the start: 2 copper layers, 15 parts, among them J1 Servo 1, J2 Servo 2, J3 Power In, J4 Prog, J5 Servo 3, U1 ATtiny404-SS, U2 AP2205-33Y-13

Commit message: more shit
Parts:
- added U3: PCF8551ATT_AJ, servo_tester:SOP50P810X120-48N, F.Cu at (156.7, 103.2)
- added U4: VIM-878-DP-FC-S-LV, servo_tester:VIM-878-DP, B.Cu at (155.7, 103.8)
- moved U1 133.1 mm to (187.4, 76.2)
- moved C2 125.0 mm to (170.0, 54.2)
- moved C3 125.0 mm to (170.0, 56.7)
- moved C4 125.0 mm to (170.0, 59.2)
- moved J1 125.0 mm to (174.5, 52.8)
- moved J2 125.0 mm to (179.1, 52.8)
- moved J4 125.0 mm to (174.5, 62.5)
- moved R1 125.0 mm to (170.0, 61.7)
- moved J3 125.0 mm to (183.7, 52.8)
- moved J5 125.0 mm to (188.3, 52.8)
- moved U2 125.0 mm to (202.0, 69.9)
- moved R2 124.1 mm to (168.9, 65.6)
- moved R3 124.1 mm to (168.9, 68.1)
- moved C1 94.2 mm to (139.0, 50.4)
- moved R4 94.2 mm to (139.0, 68.0)
Other:
- board outline added: 30 x 80 mm
