File: Electrical25-26/PCBDrone/Kicad/Kicad.kicad_pcb (KiCad board)
At the start: 2 copper layers, 35 parts, among them J1 Conn_01x02_Pin, J2 Conn_01x04, U1 ESP32-WROOM-32E, U2 BMI323, U3 DRV8210DSGR, U4 DRV8210DSGR, U5 DRV8210DSGR, U6 DRV8210DSGR

Commit message: Everything done except logo and name
Parts:
- added Motor Mount: Motor Mount, MountingHole:MotorMount, F.Cu at (95.0, 155.0)
- added Motor Mount: Motor Mount, MountingHole:MotorMount, F.Cu at (95.0, 45.0)
- added Motor Mount: Motor Mount, MountingHole:MotorMount, F.Cu at (199.8, 50.0)
- added Motor Mount: Motor Mount, MountingHole:MotorMount, F.Cu at (200.0, 150.0)
- added R8: 10k, Resistor_SMD:R_0603_1608Metric, F.Cu at (144.0, 94.0)
- added R9: 10k, Resistor_SMD:R_0603_1608Metric, F.Cu at (144.0, 96.0)
- added REF**: MountingHole_2.2mm_M2, MountingHole:MountingHole_2.2mm_M2, F.Cu at (160.0, 115.0)
- added REF**: MountingHole_2.2mm_M2, MountingHole:MountingHole_2.2mm_M2, F.Cu at (140.0, 115.0)
- added REF**: MountingHole_2.2mm_M2, MountingHole:MountingHole_2.2mm_M2, F.Cu at (160.0, 125.0)
- added REF**: MountingHole_2.2mm_M2, MountingHole:MountingHole_2.2mm_M2, F.Cu at (140.0, 125.0)
- added S2: TS04-66-50-BK-260-SMT, footprints:SW_TS04-66-50-BK-260-SMT, F.Cu at (131.6, 74.2)
- added TP1: IMU_SDA, TestPoint:TestPoint_Pad_1.0x1.0mm, F.Cu at (151.5, 94.0)
- added TP10: U3_VM, TestPoint:TestPoint_Pad_1.0x1.0mm, F.Cu at (110.0, 63.0)
- added TP11: U3_VCC, TestPoint:TestPoint_Pad_1.0x1.0mm, F.Cu at (118.5, 69.0)
- added TP12: U3_MODE, TestPoint:TestPoint_Pad_1.0x1.0mm, F.Cu at (116.5, 69.0)
- added TP13: U3_IN1, TestPoint:TestPoint_Pad_1.0x1.0mm, F.Cu at (114.5, 69.0)
- added TP14: U3_IN2, TestPoint:TestPoint_Pad_1.0x1.0mm, F.Cu at (112.5, 69.0)
- added TP15: U3_OUT1, TestPoint:TestPoint_Pad_1.0x1.0mm, F.Cu at (110.0, 65.0)
- added TP16: U3_OUT2, TestPoint:TestPoint_Pad_1.0x1.0mm, F.Cu at (110.0, 67.0)
- added TP17: U3_GND, TestPoint:TestPoint_Pad_1.0x1.0mm, F.Cu at (110.0, 69.0)
- added TP18: U4_VM, TestPoint:TestPoint_Pad_1.0x1.0mm, F.Cu at (179.5, 64.0)
- added TP19: U4_VCC, TestPoint:TestPoint_Pad_1.0x1.0mm, F.Cu at (188.0, 70.0)
- added TP2: IMU_SCL, TestPoint:TestPoint_Pad_1.0x1.0mm, F.Cu at (153.5, 94.0)
- added TP20: U4_MODE, TestPoint:TestPoint_Pad_1.0x1.0mm, F.Cu at (186.0, 70.0)
- added TP21: U4_IN1, TestPoint:TestPoint_Pad_1.0x1.0mm, F.Cu at (184.0, 70.0)
- added TP22: U4_IN2, TestPoint:TestPoint_Pad_1.0x1.0mm, F.Cu at (182.0, 70.0)
- added TP23: U4_GND, TestPoint:TestPoint_Pad_1.0x1.0mm, F.Cu at (179.5, 70.0)
- added TP24: U4_OUT1, TestPoint:TestPoint_Pad_1.0x1.0mm, F.Cu at (179.5, 66.0)
- added TP25: U4_OUT2, TestPoint:TestPoint_Pad_1.0x1.0mm, F.Cu at (179.5, 68.0)
- added TP26: U5_VM, TestPoint:TestPoint_Pad_1.0x1.0mm, F.Cu at (112.0, 130.0)
- added TP27: U5_VCC, TestPoint:TestPoint_Pad_1.0x1.0mm, F.Cu at (120.5, 136.0)
- added TP28: U5_MODE, TestPoint:TestPoint_Pad_1.0x1.0mm, F.Cu at (118.5, 136.0)
- added TP29: U5_IN1, TestPoint:TestPoint_Pad_1.0x1.0mm, F.Cu at (116.5, 136.0)
- added TP3: IMU_CSB(UNUSED), TestPoint:TestPoint_Pad_1.0x1.0mm, F.Cu at (155.5, 94.0)
- added TP30: U5_IN2, TestPoint:TestPoint_Pad_1.0x1.0mm, F.Cu at (114.5, 136.0)
- added TP31: U5_GND, TestPoint:TestPoint_Pad_1.0x1.0mm, F.Cu at (112.0, 136.0)
- added TP32: U5_OUT1, TestPoint:TestPoint_Pad_1.0x1.0mm, F.Cu at (112.0, 132.0)
- added TP33: U5_OUT2, TestPoint:TestPoint_Pad_1.0x1.0mm, F.Cu at (112.0, 134.0)
- added TP34: U6_VM, TestPoint:TestPoint_Pad_1.0x1.0mm, F.Cu at (176.5, 129.3)
- added TP35: U6_VCC, TestPoint:TestPoint_Pad_1.0x1.0mm, F.Cu at (185.0, 135.8)
- added TP36: U6_MODE, TestPoint:TestPoint_Pad_1.0x1.0mm, F.Cu at (183.0, 135.8)
- added TP37: U6_IN1, TestPoint:TestPoint_Pad_1.0x1.0mm, F.Cu at (181.0, 135.8)
- added TP38: U6_IN2, TestPoint:TestPoint_Pad_1.0x1.0mm, F.Cu at (179.0, 135.8)
- added TP39: U6_GND, TestPoint:TestPoint_Pad_1.0x1.0mm, F.Cu at (176.5, 135.3)
- added TP4: IMU_VDD, TestPoint:TestPoint_Pad_1.0x1.0mm, F.Cu at (153.5, 104.5)
- added TP40: U6_OUT1, TestPoint:TestPoint_Pad_1.0x1.0mm, F.Cu at (176.5, 131.3)
- added TP41: U6_OUT2, TestPoint:TestPoint_Pad_1.0x1.0mm, F.Cu at (176.5, 133.3)
- added TP5: IMU_INT2(UNUSED), TestPoint:TestPoint_Pad_1.0x1.0mm, F.Cu at (156.0, 100.5)
- added TP6: IMU_GND, TestPoint:TestPoint_Pad_1.0x1.0mm, F.Cu at (151.5, 105.0)
- added TP7: IMU_GNDIO, TestPoint:TestPoint_Pad_1.0x1.0mm, F.Cu at (149.5, 105.0)
- added TP8: IMU_VDDIO, TestPoint:TestPoint_Pad_1.0x1.0mm, F.Cu at (147.5, 105.0)
- added TP9: IMU_INT1(UNUSED), TestPoint:TestPoint_Pad_1.0x1.0mm, F.Cu at (145.0, 101.5)
- moved U3 120.2 mm to (115.6, 65.2)
- moved R7 92.3 mm to (126.0, 62.0)
- moved S1 91.1 mm to (131.5, 66.0)
- moved R3 89.1 mm to (120.0, 65.5), turned to 180 degrees
- moved U5 88.9 mm to (117.0, 132.5)
- moved C7 88.8 mm to (115.0, 61.5)
- moved U4 87.0 mm to (185.1, 66.2)
- moved C9 85.9 mm to (118.5, 64.0)
- moved C8 85.5 mm to (115.0, 59.5)
- moved R2 84.9 mm to (125.0, 70.0)
- moved U1 80.9 mm to (150.6, 69.5)
- moved C15 77.0 mm to (116.5, 129.0)
- moved C6 75.6 mm to (139.0, 61.5), turned to 180 degrees
- moved R5 75.5 mm to (121.7, 132.5), turned to 180 degrees
- moved U2 69.1 mm to (150.0, 100.6)
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Connections:
- R2 pad 2: Net-(U1-EN) -> Net-(R2-Pad2)
- U1 pad 13: /MOTOR1_INPUT1 -> /MOTOR4_INPUT1
- U1 pad 28: /MOTOR1_INPUT2 -> /MOTOR4_INPUT2
- U1 pad 8: /MOTOR4_INPUT1 -> /MOTOR1_INPUT1
- U1 pad 9: /MOTOR4_INPUT2 -> /MOTOR1_INPUT2
- U2 pad 12: unconnected-(U2-CSB-Pad12) -> Net-(U2-CSB)
- U2 pad 4: unconnected-(U2-INT1-Pad4) -> Net-(U2-INT1)
- U2 pad 9: unconnected-(U2-INT2-Pad9) -> Net-(U2-INT2)
Routing:
- net /VCC_3V3: track 0.00 -> 338.2 mm
- net /ESP_UART_RX: track 0.00 -> 144.1 mm, vias 0 -> 2
- net /ESP_UART_TX: track 0.00 -> 134.1 mm, vias 0 -> 2
- net /MOTOR4_INPUT1: track 0.00 -> 81.6 mm, vias 0 -> 2
- net /MOTOR4_INPUT2: track 0.00 -> 81.2 mm, vias 0 -> 2
- net /MOTOR3_INPUT1: track 0.00 -> 80.8 mm, vias 0 -> 2
- net /MOTOR3_INPUT2: track 0.00 -> 75.4 mm, vias 0 -> 2
- net /SCL: track 0.00 -> 57.0 mm, vias 0 -> 6
- net /MOTOR2_INPUT2: track 0.00 -> 53.4 mm, vias 0 -> 2
- net /SDA: track 0.00 -> 50.4 mm, vias 0 -> 6
- net /MOTOR2_INPUT1: track 0.00 -> 35.6 mm, vias 0 -> 2
- net /MOTOR1_INPUT1: track 0.00 -> 33.7 mm, vias 0 -> 2
- net /MOTOR1_INPUT2: track 0.00 -> 33.5 mm, vias 0 -> 2
- net GND: track 0.00 -> 29.7 mm, vias 0 -> 35
- net Net-(U1-EN): track 0.00 -> 29.1 mm
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- added copper zone on In2.Cu, net /VBAT
- added copper zone on In1.Cu, net GND
Other:
- board outline added: 130 x 130 mm
- copper layers 2 -> 4
- board text added: "Battery"
- board text added: "Motor 1"
- board text added: "Motor 2"
- board text added: "Motor 3"
- board text added: "Motor 4"

Commit message: Finished PCB
Parts:
- added C19: 0.1uF, Capacitor_SMD:C_0603_1608Metric, F.Cu at (162.5, 80.0)
- added C20: 0.1uF, Capacitor_SMD:C_0603_1608Metric, F.Cu at (139.0, 68.0)
- added G***: LOGO, footprints:Logo, F.Cu at (120.9, 97.9)
Connections:
- S1 pad 3: Net-(U1-SENSOR_VP) -> /BOOT
- U1 pad 25: unconnected-(U1-IO0-Pad25) -> /BOOT
- U1 pad 4: Net-(U1-SENSOR_VP) -> unconnected-(U1-SENSOR_VP-Pad4)
- U2 pad 1: unconnected-(U2-SDO-Pad1) -> GND
Routing:
- net /BOOT: track 0.00 -> 37.5 mm, vias 0 -> 2
- net Net-(U1-EN): track 29.1 -> 11.2 mm
- net /VCC_3V3: track 338.2 -> 328.9 mm
- net Net-(U1-SENSOR_VP): track 6.92 -> 0.00 mm, vias 2 -> 0
- net GND: track 29.7 -> 27.1 mm, vias 35 -> 41
- net /MOTOR3_INPUT2: track 75.4 -> 75.9 mm
Other:
- board text added: "10/21/2025"
- board text added: "BOOT"
- board text added: "EN"
- board text added: "PCB Drone v1"
- board text added: "Sreesanth Adelli"
